Commit message: 2026.10.31->配置了MBRA,准备做相机外参标定

File: src/urdf_pkg/Lite3_urdf/urdf/Lite3.urdf (robot description, URDF)
Before this commit: robot Lite3, 21 links, 20 joints
Links:
- removed link IMU_LINK
- removed link MID360_LINK
- added link camera_link
- added link imu_link
Joints:
- removed joint MID360_FIXED
- added joint D435I_TO_CAMERA_FIXED: type fixed, parent D435I_LINK, child camera_link, origin xyz=0 0 0 rpy=0 0 0
- joint D435I_FIXED: origin xyz=0.25228 -0.00050 0.07410 rpy=0 -0.3490658504 0 -> xyz=0.25489 0 0.07249 rpy=0 0.34907 0
- joint IMU_FIXED: child IMU_LINK -> imu_link; parent TORSO -> base_link
